File: rs-probe.kicad_pcb (KiCad board)
At the start: 4 copper layers, 50 x 14 mm, 120 parts, among them J1 USB_C_Receptacle_USB2.0, J10 Conn_01x01, J11 Conn_01x01, J12 Conn_01x01, J2 Conn_02x05_Odd_Even, J4 Castellated Vias, J5 tag-connect-swd, J6 Conn_01x01, J7 Conn_01x01, J8 Conn_01x01, J9 Conn_01x01, Q1 NTZD3155C, SW1 TS-1145A-C-B, SW2 TS-1145A-C-B, T1 Tab, T2 Tab, U1 74LVC1T45FZ4-7, U10 74LVC1T45FZ4-7, U11 74LVC1T45FZ4-7, U12 NCP133AMXADJTCG, U13 NCP133AMXADJTCG, U14 NCP133AMXADJTCG, U15 FM24V02A-GTR, U2 74LVC1T45FZ4-7, U3 IS25WP016D-JULE-TR, U4 NUF8401MNT4G, U5 CortexDebug, U6 RP2040, U7 NUF2042XV6T1G, U8 74LVC1T45FZ4-7, U9 74LVC1T45FZ4-7, X1 12 MHz

Commit message: 2.54mm modification.
Parts:
- moved SYM1 1.47 mm to (164.8, 97.6), turned to -170 degrees
Routing:
- net /T_TDI: track 24.8 -> 25.7 mm
- net /T_~{RESET}: track 19.1 -> 19.9 mm
- net /T_SWDCLK_JCLK: track 30.8 -> 30.1 mm
- net GND: vias 75 -> 68
Other:
- outline, holes or cut-outs redrawn
- board text added: "2.54mm Pitch version Mod from Lambda Jig"
- board text added: "20240321"
- board text removed: "20240227"
- board text removed: "Lambda Mod - SelfJig"
